File: pcb/keyplate_left.kicad_pcb (KiCad board)
At the start: 2 copper layers, 139.5 x 116.3 mm, 5 parts

Commit message: Final routing and top plates
Parts:
- moved REF** 11.4 mm to (228.8, 143.0), turned to -90 degrees
Changed lines of the file:
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@@
 	(footprint "hackbeil:logo"
 		(layer "F.Cu")
-		(at 240.125981 144.069819 -110)
+		(at 228.802268 142.985001 -90)
 		(property "Reference" "REF**"
-			(at 0 -0.500001 -110)
+			(at 0 -0.500001 -90)
 			(unlocked yes)
 			(layer "F.SilkS")
@@
 		)
 		(property "Value" "logo"
-			(at 0.000001 0.999999 -110)
+			(at 0.000001 0.999999 -90)
 			(unlocked yes)
 			(layer "F.Fab")
@@
 		)
 		(property "Footprint" "hackbeil:logo"
-			(at 0 0 -110)
+			(at 0 0 -90)
 			(unlocked yes)
 			(layer "F.Fab")
@@
 		)
 		(property "Datasheet" ""
-			(at 0 0 -110)
+			(at 0 0 -90)
 			(unlocked yes)
 			(layer "F.Fab")
@@
 		)
 		(property "Description" ""
-			(at 0 0 -110)
+			(at 0 0 -90)
 			(unlocked yes)
 			(layer "F.Fab")
@@
 		(attr smd)
 		(fp_line
+			(start 1.2 2.15)
+			(end 1.650001 2.100002)
+			(stroke
+				(width 0.2)
+				(type default)
+			)
+			(layer "F.Cu")
+		)
+		(fp_line
+			(start 1.650001 2.100002)
+			(end 1.7 1.65)
+			(stroke
+				(width 0.2)
+				(type default)
+			)
+			(layer "F.Cu")
+		)
+		(fp_line
+			(start 1.7 1.65)
+			(end 1.300001 1.625)
+			(stroke
+				(width 0.2)
+				(type default)
+			)
+			(layer "F.Cu")
+		)
+		(fp_line
+			(start 1.300001 1.625)
+			(end 1.2 2.15)
+			(stroke
+				(width 0.2)
+				(type default)
+			)
+			(layer "F.Cu")
+		)
+		(fp_line
 			(start 7.7 1.4)
 			(end 4.099999 -0.675001)
@@
 		)
 		(fp_line
-			(start 1.650001 2.100002)
-			(end 1.7 1.65)
-			(stroke
-				(width 0.2)
-				(type default)
-			)
-			(layer "F.Cu")
-		)
-		(fp_line
-			(start 1.2 2.15)
-			(end 1.650001 2.100002)
+			(start 3.8 0.9)
+			(end 4.275 0.899999)
 			(stroke
 				(width 0.2)
@@
 		)
 		(fp_line
-			(start 3.8 0.9)
-			(end 4.275 0.899999)
-			(stroke
-				(width 0.2)
-				(type default)
-			)
-			(layer "F.Cu")
-		)
-		(fp_line
-			(start 1.7 1.65)
-			(end 1.300001 1.625)
-			(stroke
-				(width 0.2)
-				(type default)
-			)
-			(layer "F.Cu")
-		)
-		(fp_line
-			(start 1.300001 1.625)
-			(end 1.2 2.15)
+			(start 3.825 0.45)
+			(end 3.8 0.9)
 			(stroke
 				(width 0.2)
@@
 		)
 		(fp_line
-			(start 3.825 0.45)
-			(end 3.8 0.9)
+			(start -0.325 -0.525)
+			(end 0.05 -0.975)
 			(stroke
 				(width 0.2)
@@
 		)
 		(fp_line
+			(start -0.775 -0.95)
+			(end -0.325 -0.525)
+			(stroke
+				(width 0.2)
+				(type default)
+			)
+			(layer "F.Cu")
+		)
+		(fp_line
+			(start 0.05 -0.975)
+			(end -0.375 -1.4)
+			(stroke
+				(width 0.2)
+				(type default)
+			)
+			(layer "F.Cu")
+		)
+		(fp_line
 			(start 2.299999 -1.024999)
 			(end 1.33 -1.455)
@@
 		)
 		(fp_line
-			(start -0.325 -0.525)
-			(end 0.05 -0.975)
+			(start -0.375 -1.4)
+			(end -0.775 -0.95)
 			(stroke
 				(width 0.2)
@@
 		)
 		(fp_line
-			(start 0.05 -0.975)
-			(end -0.375 -1.4)
+			(start -1.632499 -3.035001)
+			(end -2.717847 4.299535)
+			(stroke
+				(width 0.2)
+				(type default)
+			)
+			(layer "F.Cu")
+		)
+		(fp_line
+			(start -2.935001 -3.174999)
+			(end -4.025 4.184999)
+			(stroke
+				(width 0.2)
+				(type default)
+			)
+			(layer "F.Cu")
+		)
+		(fp_line
+			(start -3.579999 -3.205)
+			(end -3.98 -3.895)
+			(stroke
+				(width 0.2)
+				(type default)
+			)
+			(layer "F.Cu")
+		)
+		(fp_line
+			(start 5.249999 -3.7)
+			(end 5.149999 -5.499999)
 			(stroke
 				(width 0.2)
@@
 		)
 		(fp_line
-			(start -0.775 -0.95)
-			(end -0.325 -0.525)
-			(stroke
-				(width 0.2)
-				(type default)
-			)
-			(layer "F.Cu")
-		)
-		(fp_line
-			(start -0.375 -1.4)
-			(end -0.775 -0.95)
-			(stroke
-				(width 0.2)
-				(type default)
-			)
-			(layer "F.Cu")
-		)
-		(fp_line
-			(start 5.249999 -3.7)
-			(end 5.149999 -5.499999)
-			(stroke
-				(width 0.2)
-				(type default)
-			)
-			(layer "F.Cu")
-		)
-		(fp_line
 			(start 5.149999 -5.499999)
 			(end 9.475 -4.65)
@@
 		)
 		(fp_line
-			(start -1.632499 -3.035001)
-			(end -2.717847 4.299535)
-			(stroke
-				(width 0.2)
-				(type default)
-			)
-			(layer "F.Cu")
-		)
-		(fp_line
-			(start -2.935001 -3.174999)
-			(end -4.025 4.184999)
-			(stroke
-				(width 0.2)
-				(type default)
-			)
-			(layer "F.Cu")
-		)
-		(fp_line
-			(start -3.579999 -3.205)
-			(end -3.98 -3.895)
+			(start -1.132499 -6.375)
+			(end -1.0275 -6.875001)
+			(stroke
+				(width 0.2)
+				(type default)
+			)
+			(layer "F.Cu")
+		)
+		(fp_line
+			(start -2.435 -6.515)
+			(end -2.404999 -7.145001)
 			(stroke
 				(width 0.2)
@@
 		)
 		(fp_line
+			(start -3.532732 -6.713895)
+			(end -3.98 -3.895)
+			(stroke
+				(width 0.2)
+				(type default)
+			)
+			(layer "F.Cu")
+		)
+		(fp_line
+			(start 4.199999 -6.849999)
+			(end 4.574999 -6.65)
+			(stroke
+				(width 0.2)
+				(type default)
+			)
+			(layer "F.Cu")
+		)
+		(fp_line
 			(start 4.924999 -7.075001)
 			(end 4.575001 -7.350001)
@@
 		)
 		(fp_line
-			(start 4.199999 -6.849999)
-			(end 4.574999 -6.65)
-			(stroke
-				(width 0.2)
-				(type default)
-			)
-			(layer "F.Cu")
-		)
-		(fp_line
 			(start 4.575001 -7.350001)
 			(end 4.199999 -6.849999)
@@
 		)
 		(fp_line
+			(start -2.575 -7.7)
+			(end -1.740176 -6.887934)
+			(stroke
+				(width 0.2)
+				(type default)
+			)
+			(layer "F.Cu")
+		)
+		(fp_line
+			(start -2.575 -7.7)
+			(end 0.275001 -10.675)
+			(stroke
+				(width 0.2)
+				(type default)
+			)
+			(layer "F.Cu")
+		)
+		(fp_line
 			(start 3.549999 -7.974998)
 			(end 3.075 -6.125)
-			(stroke
-				(width 0.2)
-				(type default)
-			)
-			(layer "F.Cu")
-		)
-		(fp_line
-			(start -1.132499 -6.375)
-			(end -1.0275 -6.875001)
-			(stroke
-				(width 0.2)
-				(type default)
-			)
-			(layer "F.Cu")
-		)
-		(fp_line
-			(start -2.435 -6.515)
-			(end -2.404999 -7.145001)
-			(stroke
-				(width 0.2)
-				(type default)
-			)
-			(layer "F.Cu")
-		)
-		(fp_line
-			(start -3.532732 -6.713895)
-			(end -3.98 -3.895)
-			(stroke
-				(width 0.2)
-				(type default)
-			)
-			(layer "F.Cu")
-		)
-		(fp_line
-			(start -2.575 -7.7)
-			(end -1.740176 -6.887934)
-			(stroke
-				(width 0.2)
-				(type default)
-			)
-			(layer "F.Cu")
-		)
-		(fp_line
-			(start -2.575 -7.7)
-			(end 0.275001 -10.675)
 			(stroke
 				(width 0.2)
@@
 		(fp_arc
 			(start 0.500001 -2.425)
-			(mid 1.045704 -2.05184)
+			(mid 1.045705 -2.051841)
 			(end 1.329998 -1.455001)
 			(stroke
@@
 		)
 		(fp_arc
+			(start -1.0275 -6.875001)
+			(mid -1.740176 -6.887934)
+			(end -2.404999 -7.145001)
+			(stroke
+				(width 0.2)
+				(type default)
+			)
+			(layer "F.Cu")
+		)
+		(fp_arc
 			(start 2.76 -7.025001)
 			(mid 3.275914 -3.967813)
@@
 			(stroke
 				(width 0.2)
-				(type default)
-			)
-			(layer "F.Cu")
-		)
-		(fp_arc
-			(start -1.0275 -6.875001)
-			(mid -1.740176 -6.887934)
-			(end -2.404999 -7.145001)
-			(stroke
-				(width 0.2)
