File: pcb/keyplate_right.kicad_pcb (KiCad board)
At the start: 2 copper layers, 139.5 x 116.3 mm, 5 parts

Commit message: Final routing and top plates
Parts:
- moved REF** 8.57 mm to (228.8, 148.3), turned to 90 degrees
Routing:
- removed copper zone on F.Cu, net GND
